Commit message: Changed the name of the body in the slider-block's urdf. Also, added some basic floor stuff and more complex functions to the BlockHandlerSystem.

File: drake/manip_tests/slider/slider-block.urdf (robot description, URDF)
Before this commit: robot slider, 1 links, 0 joints
Links:
- removed link base
- added link body, mass 0.77; collision mesh filename=SliderBlockv3.obj scale=0.001 0.001 0.001; visual mesh filename=SliderBlockv3.obj scale=0.001 0.001 0.001
