Commit message: Fix the paddle on the end effector connector.

File: drake/bouncing_ball/ball_model/ball.urdf (robot description, URDF)
Before this commit: robot simple_ball, 1 links, 0 joints
Links:
- link ball: geometry collision mesh filename=./ball.obj scale=0.0005 0.0005 0.0005; visual mesh filename=./ball.obj scale=0.0005 0.0005 0.0005
