Commit message: Overwrote simpleDesk mesh (removed broken one), and some organization

File: data/models/simpleDesk/simpleDesk.urdf (robot description, URDF)
Before this commit: robot simpleDesk, 1 links, 0 joints
Links:
- link simpleDesk: geometry collision mesh filename=simpleDesk2.obj scale=1 1 1; visual mesh filename=simpleDesk2.obj scale=1 1 1
